File: Glyph.kicad_pcb (KiCad board)
At the start: 2 copper layers, 85.3 x 35.3 mm, 49 parts, among them J0 Battery Pads, J1 ISP, J2 USB-Micro, J3 Screw Point 1, J4 Screw Point 2, J5 Screw Point 3, J6 Screw Point 4, SW0 RESET, SW1 UP, SW2 DOWN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

Commit message: Silkscreen
Other:
- board text added: "+3v3"
- board text added: "1"
- board text added: "GND"
- board text added: "MISO"
- board text added: "MOSI"
- board text added: "RST"
- board text added: "SCK"

Commit message: capacitor label consistency
Parts:
- C1, C12, C7: value 104 -> 0.1uF
- C13, C14: value 220 -> 22pF
- C15: value 220 -> 0.1uF
- C2, C3, C4: value 105 -> 1uF
- C5, C6: value 475 -> 4.7uF
Changed lines of the file:
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@@
       (effects (font (size 1 1) (thickness 0.15)) (justify mirror))
     )
-    (fp_text value 105 (at 0 -1.65 90) (layer B.Fab)
+    (fp_text value 1uF (at 0 -1.65 90) (layer B.Fab)
       (effects (font (size 1 1) (thickness 0.15)) (justify mirror))
     )
@@
       (effects (font (size 1 1) (thickness 0.15)) (justify mirror))
     )
-    (fp_text value 105 (at 0 -1.65 90) (layer B.Fab)
+    (fp_text value 1uF (at 0 -1.65 90) (layer B.Fab)
       (effects (font (size 1 1) (thickness 0.15)) (justify mirror))
     )
@@
       (effects (font (size 1 1) (thickness 0.15)) (justify mirror))
     )
-    (fp_text value 105 (at 0 -1.65 90) (layer B.Fab)
+    (fp_text value 1uF (at 0 -1.65 90) (layer B.Fab)
       (effects (font (size 1 1) (thickness 0.15)) (justify mirror))
     )
@@
       (effects (font (size 1 1) (thickness 0.15)) (justify mirror))
     )
-    (fp_text value 475 (at 0 -1.65 180) (layer B.Fab)
+    (fp_text value 4.7uF (at 0 -1.65 180) (layer B.Fab)
       (effects (font (size 1 1) (thickness 0.15)) (justify mirror))
     )
@@
       (effects (font (size 1 1) (thickness 0.15)) (justify mirror))
     )
-    (fp_text value 475 (at 0 -1.65 90) (layer B.Fab)
+    (fp_text value 4.7uF (at 0 -1.65 90) (layer B.Fab)
       (effects (font (size 1 1) (thickness 0.15)) (justify mirror))
     )
@@
       (effects (font (size 1 1) (thickness 0.15)))
     )
-    (fp_text value 104 (at 0 1.65 90) (layer F.Fab)
+    (fp_text value 0.1uF (at 0 1.65 90) (layer F.Fab)
       (effects (font (size 1 1) (thickness 0.15)))
     )
@@
       (effects (font (size 1 1) (thickness 0.15)))
     )
-    (fp_text value 104 (at 0 1.65 90) (layer F.Fab)
+    (fp_text value 0.1uF (at 0 1.65 90) (layer F.Fab)
       (effects (font (size 1 1) (thickness 0.15)))
     )
@@
       (effects (font (size 1 1) (thickness 0.15)) (justify mirror))
     )
-    (fp_text value 104 (at 0 -1.65 270) (layer B.Fab)
+    (fp_text value 0.1uF (at 0 -1.65 270) (layer B.Fab)
       (effects (font (size 1 1) (thickness 0.15)) (justify mirror))
     )
@@
       (effects (font (size 1 1) (thickness 0.15)) (justify mirror))
     )
-    (fp_text value 220 (at 0 -1.65 270) (layer B.Fab)
+    (fp_text value 22pF (at 0 -1.65 270) (layer B.Fab)
       (effects (font (size 1 1) (thickness 0.15)) (justify mirror))
     )
@@
       (effects (font (size 1 1) (thickness 0.15)) (justify mirror))
     )
-    (fp_text value 220 (at 0 -1.65) (layer B.Fab)
+    (fp_text value 22pF (at 0 -1.65) (layer B.Fab)
       (effects (font (size 1 1) (thickness 0.15)) (justify mirror))
     )
@@
       (effects (font (size 1 1) (thickness 0.15)) (justify mirror))
     )
-    (fp_text value 220 (at 0 -1.65 90) (layer B.Fab)
-      (effects (font (size 1 1) (thickness 0.15)) (justify mirror))
-    )
+    (fp_text value 0.1uF (at 0 -1.65 90) (layer B.Fab)
+      (effects (font (size 1 1) (thickness 0.15)) (justify mirror))
+    )

Commit message: added logo
Parts:
- added LOGO: , LOGO, F.Cu at (127.9, 117.2)
