File: glyph-isp/glyph-isp.sch (KiCad schematic (older format))
At the start: 17 parts, among them J0 ISP, J1 ISP, J2 USB-Micro, U0 ATmega16U4-MU, Y1 16MHz

Commit message: capacitor values consistent
Parts:
- C0: value 104 -> 0.1uF
- C1, C2: value 220 -> 22pF
Changed lines of the file:
@@
 P 6000 3050
 F 0 "C0" H 6115 3096 50  0000 L CNN
-F 1 "104" H 6115 3005 50  0000 L CNN
+F 1 "0.1uF" H 6115 3005 50  0000 L CNN
 F 2 "Capacitor_SMD:C_0805_2012Metric_Pad1.15x1.40mm_HandSolder" H 6038 2900 50  0001 C CNN
 F 3 "~" H 6000 3050 50  0001 C CNN
@@
 P 1950 2650
 F 0 "C1" V 1900 2750 50  0000 C CNN
-F 1 "220" V 1800 2650 50  0000 C CNN
+F 1 "22pF" V 1800 2650 50  0000 C CNN
 F 2 "Capacitor_SMD:C_0805_2012Metric_Pad1.15x1.40mm_HandSolder" H 1950 2650 50  0001 C CNN
 F 3 "~" H 1950 2650 50  0001 C CNN
@@
 P 1950 2850
 F 0 "C2" V 1900 2950 50  0000 C CNN
-F 1 "220" V 2050 2850 50  0000 C CNN
+F 1 "22pF" V 2050 2850 50  0000 C CNN
 F 2 "Capacitor_SMD:C_0805_2012Metric_Pad1.15x1.40mm_HandSolder" H 1950 2850 50  0001 C CNN
 F 3 "~" H 1950 2850 50  0001 C CNN

Commit message: reworked ISP size
Changed lines of the file:
@@
 	1    0    0    -1
 $EndComp
-Text GLabel 3800 3350 2    50   Input ~ 0
+Text GLabel 3800 4050 2    50   Input ~ 0
 TARGET_RESET
 Text GLabel 5950 4800 0    50   Input ~ 0
